File: hardware/project-MS88SF3-breakout.sch (KiCad schematic (older format))
At the start: 1 part

Commit message: Most components added to schematic
Parts:
- added C? (x3): 100nF, Capacitor_SMD:C_0603_1608Metric, symbol Device:C
- added C? (x2): 4.7uF, Capacitor_SMD:C_0805_2012Metric, symbol Device:C
- added D?: LED, LED_SMD:LED_0603_1608Metric, symbol Device:LED
- added H? (x4): MountingHole_Pad, MountingHole:MountingHole_2.2mm_M2_ISO7380_Pad, symbol Mechanical:MountingHole_Pad
- added J?: USB4105-GF-A, GCT_USB4105-GF-A, symbol USB4105-GF-A:USB4105-GF-A
- added J?: SM04B-SRSS-TB(LF)(SN), JST_SM04B-SRSS-TB(LF)(SN), symbol SM04B-SRSS-TB_LF__SN_:SM04B-SRSS-TB(LF)(SN)
- added J?: Conn_02x05_Odd_Even, Connector_PinHeader_1.27mm:PinHeader_2x05_P1.27mm_Vertical_SMD, symbol Connector_Generic:Conn_02x05_Odd_Even
- added JP?: SolderJumper_2_Bridged, Jumper:SolderJumper-2_P1.3mm_Bridged_RoundedPad1.0x1.5mm, symbol Jumper:SolderJumper_2_Bridged
- added JP?: SolderJumper_2_Open, Jumper:SolderJumper-2_P1.3mm_Open_RoundedPad1.0x1.5mm, symbol Jumper:SolderJumper_2_Open
- added L?: 10uH, Inductor_SMD:L_0603_1608Metric, symbol Device:L
- added R? (x3): 5.1k, Resistor_SMD:R_0603_1608Metric, symbol Device:R
- added R?: 4.7, Resistor_SMD:R_0603_1608Metric, symbol Device:R
- added R? (x2): 22, Resistor_SMD:R_0603_1608Metric, symbol Device:R
- added R?: 1k, Resistor_SMD:R_0603_1608Metric, symbol Device:R
- added SW?: SW_SPST, Button_Switch_SMD:SW_SPST_B3U-3000P-B, symbol Switch:SW_SPST
Connections:
- net labels added: DCCH, GND, RESET, RX, TX, VBUS_CONN, VBUS_nRF, VDD_OUT
- wire segments 0 -> 22

Commit message: First placement
Parts:
- added J4: Conn_01x06_Male, Connector_PinHeader_2.54mm:PinHeader_1x06_P2.54mm_Vertical, symbol Connector:Conn_01x06_Male
- added J5: Conn_01x08_Male, Connector_PinHeader_2.54mm:PinHeader_1x08_P2.54mm_Vertical, symbol Connector:Conn_01x08_Male
- gave numbers to parts that had none: 25
Changed lines of the file:
@@
 $EndDescr
 $Comp
-L MS88SF3:MS88SF3 U?
+L MS88SF3:MS88SF3 U1
 U 1 1 62BF0ECE
 P 2700 2850
-F 0 "U?" H 2700 4717 50  0000 C CNN
+F 0 "U1" H 2700 4717 50  0000 C CNN
 F 1 "MS88SF3" H 2700 4626 50  0000 C CNN
 F 2 "MODULE_MS88SF3" H 2700 2850 50  0001 L BNN
@@
 $EndComp
 $Comp
-L power:GND #PWR?
+L power:GND #PWR01
 U 1 1 6301553B
 P 3950 4500
-F 0 "#PWR?" H 3950 4250 50  0001 C CNN
+F 0 "#PWR01" H 3950 4250 50  0001 C CNN
 F 1 "GND" H 3955 4327 50  0000 C CNN
 F 2 "" H 3950 4500 50  0001 C CNN
@@
 	3950 4450 3900 4450
 $Comp
-L USB4105-GF-A:USB4105-GF-A J?
+L USB4105-GF-A:USB4105-GF-A J3
 U 1 1 63016D79
 P 9750 1750
-F 0 "J?" H 9750 2417 50  0000 C CNN
+F 0 "J3" H 9750 2417 50  0000 C CNN
 F 1 "USB4105-GF-A" H 9750 2326 50  0000 C CNN
 F 2 "GCT_USB4105-GF-A" H 9750 1750 50  0001 L BNN
@@
 $EndComp
 $Comp
-L Device:R R?
+L Device:R R4
 U 1 1 6301B6C4
 P 8300 1500
-F 0 "R?" H 8370 1546 50  0000 L CNN
+F 0 "R4" H 8370 1546 50  0000 L CNN
 F 1 "5.1k" H 8370 1455 50  0000 L CNN
 F 2 "Resistor_SMD:R_0603_1608Metric" V 8230 1500 50  0001 C CNN
@@
 $EndComp
 $Comp
-L Device:R R?
+L Device:R R5
 U 1 1 6301BD36
 P 8600 1500
-F 0 "R?" H 8670 1546 50  0000 L CNN
+F 0 "R5" H 8670 1546 50  0000 L CNN
 F 1 "5.1k" H 8670 1455 50  0000 L CNN
 F 2 "Resistor_SMD:R_0603_1608Metric" V 8530 1500 50  0001 C CNN
@@
 $EndComp
 $Comp
-L power:GND #PWR?
+L power:GND #PWR02
 U 1 1 6301EFF7
 P 10750 2200
-F 0 "#PWR?" H 10750 1950 50  0001 C CNN
+F 0 "#PWR02" H 10750 1950 50  0001 C CNN
 F 1 "GND" H 10755 2027 50  0000 C CNN
 F 2 "" H 10750 2200 50  0001 C CNN
@@
 $EndComp
 $Comp
-L Device:L L?
+L Device:L L1
 U 1 1 630235F3
 P 4800 1100
-F 0 "L?" V 4990 1100 50  0000 C CNN
+F 0 "L1" V 4990 1100 50  0000 C CNN
 F 1 "10uH" V 4899 1100 50  0000 C CNN
 F 2 "Inductor_SMD:L_0603_1608Metric" H 4800 1100 50  0001 C CNN
@@
 	5050 1100 4950 1100
 $Comp
-L Device:R R?
+L Device:R R3
 U 1 1 630309A2
 P 5000 1950
-F 0 "R?" V 5207 1950 50  0000 C CNN
+F 0 "R3" V 5207 1950 50  0000 C CNN
 F 1 "4.7" V 5116 1950 50  0000 C CNN
 F 2 "Resistor_SMD:R_0603_1608Metric" V 4930 1950 50  0001 C CNN
@@
 	5150 1950 5650 1950
 $Comp
-L Jumper:SolderJumper_2_Bridged JP?
+L Jumper:SolderJumper_2_Bridged JP1
 U 1 1 63036196
 P 5400 1450
-F 0 "JP?" H 5400 1655 50  0000 C CNN
+F 0 "JP1" H 5400 1655 50  0000 C CNN
 F 1 "SolderJumper_2_Bridged" H 5400 1564 50  0000 C CNN
 F 2 "Jumper:SolderJumper-2_P1.3mm_Bridged_RoundedPad1.0x1.5mm" H 5400 1450 50  0001 C CNN
@@
 $EndComp
 $Comp
-L Jumper:SolderJumper_2_Open JP?
+L Jumper:SolderJumper_2_Open JP2
 U 1 1 63036BBA
 P 5650 1200
-F 0 "JP?" V 5604 1268 50  0000 L CNN
+F 0 "JP2" V 5604 1268 50  0000 L CNN
 F 1 "SolderJumper_2_Open" V 5695 1268 50  0000 L CNN
 F 2 "Jumper:SolderJumper-2_P1.3mm_Open_RoundedPad1.0x1.5mm" H 5650 1200 50  0001 C CNN
@@
 Connection ~ 5050 1250
 $Comp
-L Device:R R?
+L Device:R R6
 U 1 1 6304D352
 P 8600 2150
-F 0 "R?" V 8393 2150 50  0000 C CNN
+F 0 "R6" V 8393 2150 50  0000 C CNN
 F 1 "22" V 8484 2150 50  0000 C CNN
 F 2 "Resistor_SMD:R_0603_1608Metric" V 8530 2150 50  0001 C CNN
@@
 $EndComp
 $Comp
-L Device:R R?
+L Device:R R7
 U 1 1 6304E3E8
 P 8600 2500
-F 0 "R?" V 8393 2500 50  0000 C CNN
+F 0 "R7" V 8393 2500 50  0000 C CNN
 F 1 "22" V 8484 2500 50  0000 C CNN
 F 2 "Resistor_SMD:R_0603_1608Metric" V 8530 2500 50  0001 C CNN
@@
 $EndComp
 $Comp
-L SM04B-SRSS-TB_LF__SN_:SM04B-SRSS-TB(LF)(SN) J?
+L SM04B-SRSS-TB_LF__SN_:SM04B-SRSS-TB(LF)(SN) J2
 U 1 1 630517DF
 P 7550 4950
-F 0 "J?" H 7780 4946 50  0000 L CNN
+F 0 "J2" H 7780 4946 50  0000 L CNN
 F 1 "SM04B-SRSS-TB(LF)(SN)" H 7780 4855 50  0000 L CNN
 F 2 "JST_SM04B-SRSS-TB(LF)(SN)" H 7550 4950 50  0001 L BNN
@@
 RESET
 $Comp
-L Device:R R?
+L Device:R R1
 U 1 1 630544FE
 P 1750 5350
-F 0 "R?" H 1820 5396 50  0000 L CNN
+F 0 "R1" H 1820 5396 50  0000 L CNN
 F 1 "5.1k" H 1820 5305 50  0000 L CNN
 F 2 "Resistor_SMD:R_0603_1608Metric" V 1680 5350 50  0001 C CNN
@@
 $EndComp
 $Comp
-L Device:C C?
+L Device:C C1
 U 1 1 63054C5D
 P 1750 6000
-F 0 "C?" H 1865 6046 50  0000 L CNN
+F 0 "C1" H 1865 6046 50  0000 L CNN
 F 1 "100nF" H 1865 5955 50  0000 L CNN
 F 2 "Capacitor_SMD:C_0603_1608Metric" H 1788 5850 50  0001 C CNN
@@
 VDD_OUT
 $Comp
-L Device:LED D?
+L Device:LED D1
 U 1 1 6306A63F
 P 4450 6400
-F 0 "D?" H 4443 6145 50  0000 C CNN
+F 0 "D1" H 4443 6145 50  0000 C CNN
 F 1 "LED" H 4443 6236 50  0000 C CNN
 F 2 "LED_SMD:LED_0603_1608Metric" H 4450 6400 50  0001 C CNN
@@
 $EndComp
 $Comp
-L Device:R R?
+L Device:R R2
 U 1 1 6306BDDD
 P 3950 6400
-F 0 "R?" V 3743 6400 50  0000 C CNN
+F 0 "R2" V 3743 6400 50  0000 C CNN
 F 1 "1k" V 3834 6400 50  0000 C CNN
 F 2 "Resistor_SMD:R_0603_1608Metric" V 3880 6400 50  0001 C CNN
@@
 $EndComp
 $Comp
-L Connector_Generic:Conn_02x05_Odd_Even J?
+L Connector_Generic:Conn_02x05_Odd_Even J1
 U 1 1 63072B34
 P 7400 3750
-F 0 "J?" H 7450 4167 50  0000 C CNN
+F 0 "J1" H 7450 4167 50  0000 C CNN
 F 1 "Conn_02x05_Odd_Even" H 7450 4076 50  0000 C CNN
 F 2 "Connector_PinHeader_1.27mm:PinHeader_2x05_P1.27mm_Vertical_SMD" H 7400 3750 50  0001 C CNN
@@
 $EndComp
 $Comp
-L Device:C C?
+L Device:C C5
 U 1 1 6307991A
 P 11050 1450
-F 0 "C?" H 11165 1496 50  0000 L CNN
+F 0 "C5" H 11165 1496 50  0000 L CNN
 F 1 "100nF" H 11165 1405 50  0000 L CNN
 F 2 "Capacitor_SMD:C_0603_1608Metric" H 11088 1300 50  0001 C CNN
@@
 $EndComp
 $Comp
-L Device:C C?
+L Device:C C4
 U 1 1 6307AB03
 P 10650 1450
-F 0 "C?" H 10765 1496 50  0000 L CNN
+F 0 "C4" H 10765 1496 50  0000 L CNN
 F 1 "4.7uF" H 10765 1405 50  0000 L CNN
 F 2 "Capacitor_SMD:C_0805_2012Metric" H 10688 1300 50  0001 C CNN
@@
 $EndComp
 $Comp
-L Switch:SW_SPST SW?
+L Switch:SW_SPST SW1
 U 1 1 63080A63
 P 2300 5650
-F 0 "SW?" H 2300 5885 50  0000 C CNN
+F 0 "SW1" H 2300 5885 50  0000 C CNN
 F 1 "SW_SPST" H 2300 5794 50  0000 C CNN
 F 2 "Button_Switch_SMD:SW_SPST_B3U-3000P-B" H 2300 5650 50  0001 C CNN
@@
 $EndComp
 $Comp
-L Mechanical:MountingHole_Pad H?
+L Mechanical:MountingHole_Pad H1
 U 1 1 63082A94
 P 9550 4150
-F 0 "H?" H 9650 4199 50  0000 L CNN
+F 0 "H1" H 9650 4199 50  0000 L CNN
 F 1 "MountingHole_Pad" H 9650 4108 50  0000 L CNN
 F 2 "MountingHole:MountingHole_2.2mm_M2_ISO7380_Pad" H 9550 4150 50  0001 C CNN
@@
 $EndComp
 $Comp
-L Mechanical:MountingHole_Pad H?
+L Mechanical:MountingHole_Pad H3
 U 1 1 6308334E
 P 9900 4150
-F 0 "H?" H 10000 4199 50  0000 L CNN
+F 0 "H3" H 10000 4199 50  0000 L CNN
 F 1 "MountingHole_Pad" H 10000 4108 50  0000 L CNN
 F 2 "MountingHole:MountingHole_2.2mm_M2_ISO7380_Pad" H 9900 4150 50  0001 C CNN
@@
 $EndComp
 $Comp
-L Mechanical:MountingHole_Pad H?
+L Mechanical:MountingHole_Pad H2
 U 1 1 63083EDA
 P 9550 4500
-F 0 "H?" H 9650 4549 50  0000 L CNN
+F 0 "H2" H 9650 4549 50  0000 L CNN
 F 1 "MountingHole_Pad" H 9650 4458 50  0000 L CNN
 F 2 "MountingHole:MountingHole_2.2mm_M2_ISO7380_Pad" H 9550 4500 50  0001 C CNN
@@
 $EndComp
 $Comp
-L Mechanical:MountingHole_Pad H?
+L Mechanical:MountingHole_Pad H4
 U 1 1 63083EE0
 P 9900 4500
-F 0 "H?" H 10000 4549 50  0000 L CNN
+F 0 "H4" H 10000 4549 50  0000 L CNN
 F 1 "MountingHole_Pad" H 10000 4458 50  0000 L CNN
 F 2 "MountingHole:MountingHole_2.2mm_M2_ISO7380_Pad" H 9900 4500 50  0001 C CNN
@@
 $EndComp
 $Comp
-L Device:C C?
+L Device:C C3
 U 1 1 63088C20
 P 6150 800
-F 0 "C?" H 6265 846 50  0000 L CNN
+F 0 "C3" H 6265 846 50  0000 L CNN
 F 1 "100nF" H 6265 755 50  0000 L CNN
 F 2 "Capacitor_SMD:C_0603_1608Metric" H 6188 650 50  0001 C CNN
@@
 $EndComp
 $Comp
-L Device:C C?
+L Device:C C2
 U 1 1 63088C26
 P 5750 800
-F 0 "C?" H 5865 846 50  0000 L CNN
+F 0 "C2" H 5865 846 50  0000 L CNN
 F 1 "4.7uF" H 5865 755 50  0000 L CNN
 F 2 "Capacitor_SMD:C_0805_2012Metric" H 5788 650 50  0001 C CNN
@@
 	1    0    0    -1
 $EndComp
+$Comp
+L Connector:Conn_01x06_Male J4
+U 1 1 6309BC95
+P 4900 4300
+F 0 "J4" H 5008 4681 50  0000 C CNN
+F 1 "Conn_01x06_Male" H 5008 4590 50  0000 C CNN
+F 2 "Connector_PinHeader_2.54mm:PinHeader_1x06_P2.54mm_Vertical" H 4900 4300 50  0001 C CNN
+F 3 "~" H 4900 4300 50  0001 C CNN
+	1    4900 4300
+	1    0    0    -1
+$EndComp
+$Comp
+L Connector:Conn_01x08_Male J5
+U 1 1 6309C92F
+P 5550 4350
+F 0 "J5" H 5658 4831 50  0000 C CNN
+F 1 "Conn_01x08_Male" H 5658 4740 50  0000 C CNN
+F 2 "Connector_PinHeader_2.54mm:PinHeader_1x08_P2.54mm_Vertical" H 5550 4350 50  0001 C CNN
+F 3 "~" H 5550 4350 50  0001 C CNN
+	1    5550 4350
+	1    0    0    -1
+$EndComp

Commit message: Add wires to schematic
Parts:
- removed J2: SM04B-SRSS-TB(LF)(SN), JST_SM04B-SRSS-TB(LF)(SN), symbol SM04B-SRSS-TB_LF__SN_:SM04B-SRSS-TB(LF)(SN)
Connections:
- net labels added: CC1, CC2, D+, D-, D_N, D_P, SWCLK, SWDIO, VBUS, VDDH, VDD_nRF
- net labels removed: VBUS_CONN, VDD_OUT
- wire segments 22 -> 90
- no-connect marks 0 -> 2
Other:
- note added: "(VDD OUT)"
- moved on the sheet: C1, C2, C3, C4, C5, D1, H1, H2, H3, H4, J1, J3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

Commit message: Make it a feather shape
Parts:
- removed SW1: SW_SPST, Button_Switch_SMD:SW_SPST_B3U-3000P-B, symbol Switch:SW_SPST
- added J2: S2B-PH-SM4-TB(LF)(SN), JST_S2B-PH-SM4-TB(LF)(SN), symbol S2B-PH-SM4-TB_LF__SN_:S2B-PH-SM4-TB(LF)(SN)
- added S1: 435151014824, 435151014824, symbol 435151014824:435151014824
- J4: value Conn_01x06_Male -> Conn_01x12_Male; footprint Connector_PinHeader_2.54mm:PinHeader_1x06_P2.54mm_Vertical -> Connector_PinHeader_2.54mm:PinHeader_1x12_P2.54mm_Vertical; symbol Connector:Conn_01x06_Male -> Connector:Conn_01x12_Male
- J5: value Conn_01x08_Male -> Conn_01x16_Male; footprint Connector_PinHeader_2.54mm:PinHeader_1x08_P2.54mm_Vertical -> Connector_PinHeader_2.54mm:PinHeader_1x16_P2.54mm_Vertical; symbol Connector:Conn_01x08_Male -> Connector:Conn_01x16_Male
Connections:
- wire segments 90 -> 104
Other:
- moved on the sheet: H2, H3
Changed lines of the file:
@@
-$EndComp
-$Comp
-L Switch:SW_SPST SW1
-U 1 1 63080A63
-P 2250 5600
-F 0 "SW1" H 2250 5835 50  0000 C CNN
-F 1 "SW_SPST" H 2250 5744 50  0000 C CNN
-F 2 "Button_Switch_SMD:SW_SPST_B3U-3000P-B" H 2250 5600 50  0001 C CNN
-F 3 "~" H 2250 5600 50  0001 C CNN
-	1    2250 5600
-	1    0    0    -1
 $EndComp
 $Comp
@@
 U 1 1 63082A94
 P 10050 5300
-F 0 "H1" H 10150 5349 50  0000 L CNN
-F 1 "MountingHole_Pad" H 10150 5258 50  0000 L CNN
+F 0 "H1" H 10150 5303 50  0000 L CNN
+F 1 "MountingHole_Pad" H 10150 5258 50  0001 L CNN
 F 2 "MountingHole:MountingHole_2.2mm_M2_ISO7380_Pad" H 10050 5300 50  0001 C CNN
 F 3 "~" H 10050 5300 50  0001 C CNN
@@
 L Mechanical:MountingHole_Pad H3
 U 1 1 6308334E
+P 10050 5900
+F 0 "H3" H 10150 5949 50  0000 L CNN
+F 1 "MountingHole_Pad" H 10000 6100 50  0001 L CNN
+F 2 "MountingHole:MountingHole_2.2mm_M2_ISO7380_Pad" H 10050 5900 50  0001 C CNN
+F 3 "~" H 10050 5900 50  0001 C CNN
+	1    10050 5900
+	1    0    0    -1
+$EndComp
+$Comp
+L Mechanical:MountingHole_Pad H2
+U 1 1 63083EDA
 P 10400 5300
-F 0 "H3" H 10500 5349 50  0000 L CNN
-F 1 "MountingHole_Pad" H 10350 5500 50  0000 L CNN
+F 0 "H2" H 10500 5303 50  0000 L CNN
+F 1 "MountingHole_Pad" H 10500 5258 50  0001 L CNN
 F 2 "MountingHole:MountingHole_2.2mm_M2_ISO7380_Pad" H 10400 5300 50  0001 C CNN
 F 3 "~" H 10400 5300 50  0001 C CNN
 	1    10400 5300
-	1    0    0    -1
-$EndComp
-$Comp
-L Mechanical:MountingHole_Pad H2
-U 1 1 63083EDA
-P 10050 5900
-F 0 "H2" H 10150 5949 50  0000 L CNN
-F 1 "MountingHole_Pad" H 10150 5858 50  0000 L CNN
-F 2 "MountingHole:MountingHole_2.2mm_M2_ISO7380_Pad" H 10050 5900 50  0001 C CNN
-F 3 "~" H 10050 5900 50  0001 C CNN
-	1    10050 5900
 	1    0    0    -1
 $EndComp
@@
 P 10400 5900
 F 0 "H4" H 10500 5949 50  0000 L CNN
-F 1 "MountingHole_Pad" H 10350 6100 50  0000 L CNN
+F 1 "MountingHole_Pad" H 10350 6100 50  0001 L CNN
 F 2 "MountingHole:MountingHole_2.2mm_M2_ISO7380_Pad" H 10400 5900 50  0001 C CNN
 F 3 "~" H 10400 5900 50  0001 C CNN
@@
 $EndComp
 $Comp
-L Connector:Conn_01x06_Male J4
+L Connector:Conn_01x12_Male J4
 U 1 1 6309BC95
 P 4900 4300
-F 0 "J4" H 5008 4681 50  0000 C CNN
-F 1 "Conn_01x06_Male" H 5008 4590 50  0000 C CNN
-F 2 "Connector_PinHeader_2.54mm:PinHeader_1x06_P2.54mm_Vertical" H 4900 4300 50  0001 C CNN
+F 0 "J4" H 5008 4981 50  0000 C CNN
+F 1 "Conn_01x12_Male" H 5008 4890 50  0000 C CNN
+F 2 "Connector_PinHeader_2.54mm:PinHeader_1x12_P2.54mm_Vertical" H 4900 4300 50  0001 C CNN
 F 3 "~" H 4900 4300 50  0001 C CNN
 	1    4900 4300
@@
 $EndComp
 $Comp
-L Connector:Conn_01x08_Male J5
+L Connector:Conn_01x16_Male J5
 U 1 1 6309C92F
 P 5650 4400
-F 0 "J5" H 5758 4881 50  0000 C CNN
-F 1 "Conn_01x08_Male" H 5758 4790 50  0000 C CNN
-F 2 "Connector_PinHeader_2.54mm:PinHeader_1x08_P2.54mm_Vertical" H 5650 4400 50  0001 C CNN
+F 0 "J5" H 5758 5281 50  0000 C CNN
+F 1 "Conn_01x16_Male" H 5758 5190 50  0000 C CNN
+F 2 "Connector_PinHeader_2.54mm:PinHeader_1x16_P2.54mm_Vertical" H 5650 4400 50  0001 C CNN
 F 3 "~" H 5650 4400 50  0001 C CNN
 	1    5650 4400
@@
 VDD_nRF
 $Comp
-L power:GND #PWR?
+L power:GND #PWR0101
 U 1 1 630D786E
 P 4000 7150
-F 0 "#PWR?" H 4000 6900 50  0001 C CNN
+F 0 "#PWR0101" H 4000 6900 50  0001 C CNN
 F 1 "GND" H 4005 6977 50  0000 C CNN
 F 2 "" H 4000 7150 50  0001 C CNN
@@
 $EndComp
 $Comp
-L power:GND #PWR?
+L power:GND #PWR0102
 U 1 1 630D7CEA
-P 2650 6100
-F 0 "#PWR?" H 2650 5850 50  0001 C CNN
-F 1 "GND" H 2655 5927 50  0000 C CNN
-F 2 "" H 2650 6100 50  0001 C CNN
-F 3 "" H 2650 6100 50  0001 C CNN
-	1    2650 6100
+P 3150 6100
+F 0 "#PWR0102" H 3150 5850 50  0001 C CNN
+F 1 "GND" H 3155 5927 50  0000 C CNN
+F 2 "" H 3150 6100 50  0001 C CNN
+F 3 "" H 3150 6100 50  0001 C CNN
+	1    3150 6100
 	1    0    0    -1
 $EndComp
@@
 	1750 5600 1750 5700
 Wire Wire Line
-	2050 5600 1750 5600
-Wire Wire Line
-	2450 5600 2650 5600
-Wire Wire Line
-	2650 5600 2650 6100
+	3150 5600 3150 6100
 Text Label 8300 5350 2    50   ~ 0
 RESET
@@
 	8300 5350 7950 5350
 $Comp
-L power:GND #PWR?
+L power:GND #PWR0103
 U 1 1 630E0693
 P 7350 5400
-F 0 "#PWR?" H 7350 5150 50  0001 C CNN
+F 0 "#PWR0103" H 7350 5150 50  0001 C CNN
 F 1 "GND" H 7355 5227 50  0000 C CNN
 F 2 "" H 7350 5400 50  0001 C CNN
@@
 	7350 5350 7450 5350
 $Comp
-L power:GND #PWR?
+L power:GND #PWR0104
 U 1 1 630E24BF
 P 3950 4500
-F 0 "#PWR?" H 3950 4250 50  0001 C CNN
+F 0 "#PWR0104" H 3950 4250 50  0001 C CNN
 F 1 "GND" H 3955 4327 50  0000 C CNN
 F 2 "" H 3950 4500 50  0001 C CNN
@@
 Connection ~ 5800 1150
 $Comp
-L power:GND #PWR?
+L power:GND #PWR0105
 U 1 1 630EDA38
 P 5800 1650
-F 0 "#PWR?" H 5800 1400 50  0001 C CNN
+F 0 "#PWR0105" H 5800 1400 50  0001 C CNN
 F 1 "GND" H 5805 1477 50  0000 C CNN
 F 2 "" H 5800 1650 50  0001 C CNN
@@
 Connection ~ 10350 3800
 $Comp
-L power:GND #PWR?
+L power:GND #PWR0106
 U 1 1 630F99AF
 P 10350 4300
-F 0 "#PWR?" H 10350 4050 50  0001 C CNN
+F 0 "#PWR0106" H 10350 4050 50  0001 C CNN
 F 1 "GND" H 10355 4127 50  0000 C CNN
 F 2 "" H 10350 4300 50  0001 C CNN
@@
 	8650 3900 9250 3900
 $Comp
-L power:GND #PWR?
+L power:GND #PWR0107
 U 1 1 6315EA47
 P 8950 4500
-F 0 "#PWR?" H 8950 4250 50  0001 C CNN
+F 0 "#PWR0107" H 8950 4250 50  0001 C CNN
 F 1 "GND" H 8955 4327 50  0000 C CNN
 F 2 "" H 8950 4500 50  0001 C CNN
@@
 $EndComp
 $Comp
-L power:GND #PWR?
+L power:GND #PWR0108
 U 1 1 6315EEF7
 P 9250 4500
-F 0 "#PWR?" H 9250 4250 50  0001 C CNN
+F 0 "#PWR0108" H 9250 4250 50  0001 C CNN
 F 1 "GND" H 9255 4327 50  0000 C CNN
 F 2 "" H 9250 4500 50  0001 C CNN
@@
 NoConn ~ 9400 2900
 $Comp
-L power:GND #PWR?
+L power:GND #PWR0109
 U 1 1 63167C0C
 P 10050 6100
-F 0 "#PWR?" H 10050 5850 50  0001 C CNN
+F 0 "#PWR0109" H 10050 5850 50  0001 C CNN
 F 1 "GND" H 10055 5927 50  0000 C CNN
 F 2 "" H 10050 6100 50  0001 C CNN
@@
 	10050 6050 10050 6100
 $Comp
-L power:GND #PWR?
+L power:GND #PWR0110
 U 1 1 63173099
 P 10050 5500
-F 0 "#PWR?" H 10050 5250 50  0001 C CNN
+F 0 "#PWR0110" H 10050 5250 50  0001 C CNN
 F 1 "GND" H 10055 5327 50  0000 C CNN
 F 2 "" H 10050 5500 50  0001 C CNN
@@
 	0    -1   -1   0
 $EndComp
+$Comp
+L S2B-PH-SM4-TB_LF__SN_:S2B-PH-SM4-TB(LF)(SN) J2
+U 1 1 6322C248
+P 4750 5450
+F 0 "J2" H 4978 5446 50  0000 L CNN
+F 1 "S2B-PH-SM4-TB(LF)(SN)" H 4978 5355 50  0000 L CNN
+F 2 "JST_S2B-PH-SM4-TB(LF)(SN)" H 4750 5450 50  0001 L BNN
+F 3 "" H 4750 5450 50  0001 L BNN
+F 4 "Manufacturer Recommendation" H 4750 5450 50  0001 L BNN "STANDARD"
+F 5 "JST" H 4750 5450 50  0001 L BNN "MANUFACTURER"
+	1    4750 5450
+	1    0    0    -1
+$EndComp
+Text Label 4150 4050 2    50   ~ 0
+D_P
+Text Label 4150 4150 2    50   ~ 0
+D_N
+Wire Wire Line
+	4150 4150 3900 4150
+Wire Wire Line
+	4150 4050 3900 4050
+$Comp
+L 435151014824:435151014824 S1
+U 1 1 63271893
+P 2450 5600
+F 0 "S1" H 2450 5885 50  0000 C CNN
+F 1 "435151014824" H 2450 5794 50  0000 C CNN
+F 2 "435151014824" H 3150 5600 50  0001 L BNN
+F 3 "" H 2450 5700 50  0001 L BNN
+F 4 "435151014824" H 3150 5700 50  0001 L BNN "PART-NUMBER"
+F 5 "9500" H 2850 5600 50  0001 L BNN "QTY"
+F 6 "https://www.we-online.com/catalog/datasheet/435151014824 .pdf" H 2850 5500 50  0001 L BNN "DATASHEET-URL"
+F 7 "1.4mm" H 2850 5700 50  0001 L BNN "H"
+F 8 "240g" H 2850 5800 50  0001 L BNN "OPERATION-FORCE"
+F 9 "435151014824" H 3150 5800 50  0001 L BNN "VALUE"
+	1    2450 5600
+	1    0    0    -1
+$EndComp
+Wire Wire Line
+	1750 5600 2150 5600
+Wire Wire Line
+	2250 5700 2150 5700
+Wire Wire Line
+	2150 5700 2150 5600
+Connection ~ 2150 5600
+Wire Wire Line
+	2150 5600 2250 5600
+Wire Wire Line
+	2650 5600 2750 5600
+Wire Wire Line
+	2650 5700 2750 5700
+Wire Wire Line
+	2750 5700 2750 5600
+Connection ~ 2750 5600
+Wire Wire Line
+	2750 5600 3150 5600
+$Comp
+L power:GND #PWR03
+U 1 1 6328C2C4
+P 2750 6100
+F 0 "#PWR03" H 2750 5850 50  0001 C CNN
+F 1 "GND" H 2755 5927 50  0000 C CNN
+F 2 "" H 2750 6100 50  0001 C CNN
+F 3 "" H 2750 6100 50  0001 C CNN
+	1    2750 6100
+	1    0    0    -1
+$EndComp
+Wire Wire Line
+	2650 5800 2750 5800
+Wire Wire Line
+	2750 5800 2750 5900
+Wire Wire Line
+	2250 5800 2200 5800
+Wire Wire Line
+	2200 5800 2200 5900
+Wire Wire Line
+	2200 5900 2750 5900
+Connection ~ 2750 5900
+Wire Wire Line
+	2750 5900 2750 6100
 $EndSCHEMATC
