File: hardware/project-MS88SF3-breakout.kicad_sch (KiCad schematic)
At the start: 27 parts, among them J1 Conn_02x05_Odd_Even, J2 S2B-PH-SM4-TB(LF)(SN), J3 USB4105-GF-A, J4 Conn_01x12_Pin, J5 Conn_01x16_Pin, SW1 PTS810_SJM_250_SMTR_LFS, U1 MS88SF3_NRF52840

Commit message: Finish routing
Connections:
- net AIN4: now also J4.8 (Pin_8), U1.11 (P0.28/AIN4); no longer J4.7 (Pin_7)
- net AIN5: now also J4.7 (Pin_7)
- net AIN6: now also J4.9 (Pin_9); no longer J4.8 (Pin_8)
- net AIN7: no longer J4.9 (Pin_9)
- net NFC1: now also J5.11 (Pin_11)
- net NFC2: now also J5.12 (Pin_12)
- net P0.13: now also J5.10 (Pin_10); no longer J5.3 (Pin_3), J5.9 (Pin_9)
- net P0.15: now also J5.3 (Pin_3); no longer J5.10 (Pin_10)
- net P0.17: now also J5.9 (Pin_9); no longer J5.11 (Pin_11), J5.2 (Pin_2)
- net P0.19: no longer J5.8 (Pin_8)
- net P0.20: no longer J5.6 (Pin_6)
- net P0.21: now also J5.2 (Pin_2); no longer J5.12 (Pin_12)
- net P0.22: now also J5.7 (Pin_7); no longer J5.5 (Pin_5)
- net P0.23: now also J5.8 (Pin_8); no longer J5.7 (Pin_7)
- net P0.24: now also J5.6 (Pin_6)
- net P1.00: now reaches U1.47 (P1.00/TRACEDATA0)
- net P1.00: now also J5.5 (Pin_5)
- net P1.10: no longer names the net of U1.4 (P1.10)
- net P1.13: no longer names the net of U1.7 (P1.13)
- net P1.14: no longer names the net of U1.5 (P1.14)
- net P1.15: no longer names the net of U1.8 (P1.15)
- no-connect marks 23 -> 29
Changed lines of the file:
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@@
+	)
+	(no_connect
+		(at 91.44 114.3)
 	)
 	(no_connect
@@
 	)
 	(no_connect
-		(at 91.44 66.04)
-	)
-	(no_connect
 		(at 251.46 118.11)
 	)
@@
 	)
 	(no_connect
+		(at 91.44 96.52)
+	)
+	(no_connect
+		(at 30.48 88.9)
+	)
+	(no_connect
 		(at 91.44 81.28)
 	)
 	(no_connect
-		(at 91.44 96.52)
-	)
-	(no_connect
-		(at 30.48 88.9)
-	)
-	(no_connect
 		(at 91.44 88.9)
 	)
 	(no_connect
+		(at 21.59 66.04)
+	)
+	(no_connect
 		(at 30.48 93.98)
 	)
 	(no_connect
+		(at 91.44 104.14)
+	)
+	(no_connect
 		(at 210.82 118.11)
 	)
 	(no_connect
+		(at 21.59 63.5)
+	)
+	(no_connect
 		(at 137.16 54.61)
 	)
@@
 	)
 	(no_connect
+		(at 91.44 111.76)
+	)
+	(no_connect
 		(at 91.44 91.44)
 	)
@@
 	)
 	(no_connect
+		(at 91.44 116.84)
+	)
+	(no_connect
+		(at 100.33 58.42)
+	)
+	(no_connect
+		(at 30.48 86.36)
+	)
+	(no_connect
+		(at 30.48 45.72)
+	)
+	(no_connect
+		(at 91.44 99.06)
+	)
+	(no_connect
+		(at 100.33 73.66)
+	)
+	(no_connect
 		(at 91.44 86.36)
 	)
-	(no_connect
-		(at 91.44 78.74)
-	)
-	(no_connect
-		(at 30.48 86.36)
-	)
-	(no_connect
-		(at 30.48 45.72)
-	)
-	(no_connect
-		(at 91.44 99.06)
-	)
 	(wire
 		(pts
@@
 	(wire
 		(pts
-			(xy 100.33 104.14) (xy 91.44 104.14)
-		)
-		(stroke
-			(width 0)
-			(type default)
-		)
-	)
-	(wire
-		(pts
 			(xy 161.29 41.91) (xy 152.4 41.91)
 		)
@@
 	(wire
 		(pts
-			(xy 100.33 116.84) (xy 91.44 116.84)
+			(xy 100.33 66.04) (xy 91.44 66.04)
 		)
 		(stroke
@@
 	(wire
 		(pts
-			(xy 100.33 111.76) (xy 91.44 111.76)
-		)
-		(stroke
-			(width 0)
-			(type default)
-		)
-	)
-	(wire
-		(pts
-			(xy 100.33 114.3) (xy 91.44 114.3)
-		)
-		(stroke
-			(width 0)
-			(type default)
-		)
-	)
-	(wire
-		(pts
 			(xy 133.35 115.57) (xy 142.24 115.57)
 		)
@@
 		(pts
 			(xy 46.99 177.8) (xy 46.99 180.34)
+		)
+		(stroke
+			(width 0)
+			(type default)
+		)
+	)
+	(wire
+		(pts
+			(xy 100.33 78.74) (xy 91.44 78.74)
 		)
 		(stroke
@@
 		)
 	)
-	(label "P0.21"
+	(label "NFC2"
 		(at 152.4 57.15 0)
 		(fields_autoplaced yes)
@@
 		)
 	)
-	(label "P0.22"
+	(label "P1.00"
 		(at 152.4 39.37 0)
 		(fields_autoplaced yes)
@@
 		)
 	)
-	(label "P1.15"
-		(at 100.33 116.84 180)
-		(fields_autoplaced yes)
-		(effects
-			(font
-				(size 1.27 1.27)
-			)
-			(justify right bottom)
-		)
-	)
-	(label "AIN6"
+	(label "AIN4"
 		(at 128.27 46.99 0)
 		(fields_autoplaced yes)
@@
 			)
 			(justify left bottom)
+		)
+	)
+	(label "P1.00"
+		(at 100.33 78.74 180)
+		(fields_autoplaced yes)
+		(effects
+			(font
+				(size 1.27 1.27)
+			)
+			(justify right bottom)
 		)
 	)
@@
 		)
 	)
-	(label "P0.13"
+	(label "P0.15"
 		(at 152.4 34.29 0)
 		(fields_autoplaced yes)
@@
 		)
 	)
-	(label "P0.17"
+	(label "NFC1"
 		(at 152.4 54.61 0)
 		(fields_autoplaced yes)
@@
 		)
 	)
-	(label "P0.13"
+	(label "P0.17"
 		(at 152.4 49.53 0)
 		(fields_autoplaced yes)
@@
 		)
 	)
-	(label "P0.17"
+	(label "P0.21"
 		(at 152.4 31.75 0)
 		(fields_autoplaced yes)
@@
 		)
 	)
-	(label "P1.13"
-		(at 100.33 111.76 180)
-		(fields_autoplaced yes)
-		(effects
-			(font
-				(size 1.27 1.27)
-			)
-			(justify right bottom)
-		)
-	)
 	(label "VDD_nRF"
 		(at 185.42 71.12 0)
@@
 		)
 	)
-	(label "P0.15"
+	(label "P0.13"
 		(at 152.4 52.07 0)
 		(fields_autoplaced yes)
@@
 		)
 	)
-	(label "P0.19"
+	(label "P0.23"
 		(at 152.4 46.99 0)
 		(fields_autoplaced yes)
@@
 		)
 	)
-	(label "P1.14"
-		(at 100.33 114.3 180)
-		(fields_autoplaced yes)
-		(effects
-			(font
-				(size 1.27 1.27)
-			)
-			(justify right bottom)
-		)
-	)
 	(label "P0.19"
 		(at 21.59 106.68 0)
@@
 		)
 	)
-	(label "AIN7"
+	(label "AIN6"
 		(at 128.27 49.53 0)
 		(fields_autoplaced yes)
@@
 		)
 	)
+	(label "AIN4"
+		(at 100.33 66.04 180)
+		(fields_autoplaced yes)
+		(effects
+			(font
+				(size 1.27 1.27)
+			)
+			(justify right bottom)
+		)
+	)
 	(label "D_N"
 		(at 212.09 148.59 180)
@@
 		)
 	)
-	(label "P0.23"
+	(label "P0.22"
 		(at 152.4 44.45 0)
 		(fields_autoplaced yes)
@@
 		)
 	)
-	(label "P1.10"
-		(at 100.33 104.14 180)
-		(fields_autoplaced yes)
-		(effects
-			(font
-				(size 1.27 1.27)
-			)
-			(justify right bottom)
-		)
-	)
-	(label "P0.20"
+	(label "P0.24"
 		(at 152.4 41.91 0)
 		(fields_autoplaced yes)
@@
 		)
 	)
-	(label "AIN4"
+	(label "AIN5"
 		(at 128.27 44.45 0)
 		(fields_autoplaced yes)
